File: shield MCU/shield MCU/shield MCU V2.kicad_sch (KiCad schematic)
At the start: 16 parts, among them J1 IR_sensor, J2 IR_sensor, J3 IR_sensor, J4 IR_sensor, J5 IR_sensor, J6 BATT, SW1 Pwr_Sw, U1 pwr_mgr_1, U3 gy50, U4 NUCLEO144-F429ZI

Commit message: uusi pcb
Connections:
- no-connect marks 2 -> 1
Other:
- moved on the sheet: J5
Changed lines of the file:
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@@
 (kicad_sch (version 20211123) (generator eeschema)
   (paper "A3")
-  (junction (at 124.46 50.8) (diameter 0) (color 0 0 0 0)
+  (junction (at 294.64 177.8) (diameter 0) (color 0 0 0 0)
   )
   (junction (at 73.66 144.78) (diameter 0) (color 0 0 0 0)
   )
+  (junction (at 168.91 46.99) (diameter 0) (color 0 0 0 0)
+  )
   (junction (at 299.72 157.48) (diameter 0) (color 0 0 0 0)
   )
@@
   (junction (at 71.12 163.83) (diameter 0) (color 0 0 0 0)
   )
-  (junction (at 109.22 34.29) (diameter 0) (color 0 0 0 0)
-  )
   (junction (at 171.45 44.45) (diameter 0) (color 0 0 0 0)
   )
@@
   (junction (at 144.78 251.46) (diameter 0) (color 0 0 0 0)
   )
-  (junction (at 168.91 50.8) (diameter 0) (color 0 0 0 0)
-  )
   (junction (at 294.64 148.59) (diameter 0) (color 0 0 0 0)
   )
   (junction (at 38.1 36.83) (diameter 0) (color 0 0 0 0)
   )
+  (junction (at 299.72 175.26) (diameter 0) (color 0 0 0 0)
+  )
   (no_connect (at 88.9 20.32))
-  (no_connect (at 109.22 20.32))
   (wire (pts (xy 231.14 208.28) (xy 240.03 208.28))
     (stroke (width 0) (type default) (color 0 0 0 0))
@@
     (stroke (width 0) (type default) (color 0 0 0 0))
   )
-  (wire (pts (xy 124.46 50.8) (xy 168.91 50.8))
-    (stroke (width 0) (type default) (color 0 0 0 0))
-  )
   (wire (pts (xy 303.53 154.94) (xy 209.55 154.94))
     (stroke (width 0) (type default) (color 0 0 0 0))
@@
     (stroke (width 0) (type default) (color 0 0 0 0))
   )
-  (wire (pts (xy 294.64 160.02) (xy 294.64 195.58))
-    (stroke (width 0) (type default) (color 0 0 0 0))
-  )
   (wire (pts (xy 77.47 20.32) (xy 86.36 20.32))
     (stroke (width 0) (type default) (color 0 0 0 0))
@@
     (stroke (width 0) (type default) (color 0 0 0 0))
   )
+  (wire (pts (xy 288.29 157.48) (xy 212.09 157.48))
+    (stroke (width 0) (type default) (color 0 0 0 0))
+  )
   (wire (pts (xy 294.64 160.02) (xy 303.53 160.02))
     (stroke (width 0) (type default) (color 0 0 0 0))
@@
     (stroke (width 0) (type default) (color 0 0 0 0))
   )
-  (wire (pts (xy 124.46 46.99) (xy 124.46 50.8))
+  (wire (pts (xy 168.91 46.99) (xy 168.91 55.88))
     (stroke (width 0) (type default) (color 0 0 0 0))
   )
@@
     (stroke (width 0) (type default) (color 0 0 0 0))
   )
-  (wire (pts (xy 121.92 53.34) (xy 129.54 53.34))
+  (wire (pts (xy 299.72 175.26) (xy 299.72 184.15))
     (stroke (width 0) (type default) (color 0 0 0 0))
   )
@@
     (stroke (width 0) (type default) (color 0 0 0 0))
   )
+  (wire (pts (xy 294.64 177.8) (xy 294.64 195.58))
+    (stroke (width 0) (type default) (color 0 0 0 0))
+  )
   (wire (pts (xy 299.72 157.48) (xy 303.53 157.48))
     (stroke (width 0) (type default) (color 0 0 0 0))
@@
     (stroke (width 0) (type default) (color 0 0 0 0))
   )
-  (wire (pts (xy 80.01 34.29) (xy 109.22 34.29))
+  (wire (pts (xy 80.01 34.29) (xy 115.57 34.29))
     (stroke (width 0) (type default) (color 0 0 0 0))
   )
@@
     (stroke (width 0) (type default) (color 0 0 0 0))
   )
+  (wire (pts (xy 191.77 179.07) (xy 212.09 179.07))
+    (stroke (width 0) (type default) (color 0 0 0 0))
+  )
   (wire (pts (xy 234.95 228.6) (xy 234.95 213.36))
     (stroke (width 0) (type default) (color 0 0 0 0))
@@
     (stroke (width 0) (type default) (color 0 0 0 0))
   )
-  (wire (pts (xy 194.31 54.61) (xy 194.31 179.07))
+  (wire (pts (xy 299.72 175.26) (xy 303.53 175.26))
     (stroke (width 0) (type default) (color 0 0 0 0))
   )
@@
     (stroke (width 0) (type default) (color 0 0 0 0))
   )
-  (wire (pts (xy 121.92 58.42) (xy 121.92 55.88))
-    (stroke (width 0) (type default) (color 0 0 0 0))
-  )
   (wire (pts (xy 281.94 200.66) (xy 281.94 246.38))
     (stroke (width 0) (type default) (color 0 0 0 0))
@@
     (stroke (width 0) (type default) (color 0 0 0 0))
   )
-  (wire (pts (xy 194.31 179.07) (xy 191.77 179.07))
+  (wire (pts (xy 212.09 157.48) (xy 212.09 179.07))
     (stroke (width 0) (type default) (color 0 0 0 0))
   )
@@
     (stroke (width 0) (type default) (color 0 0 0 0))
   )
-  (wire (pts (xy 105.41 46.99) (xy 124.46 46.99))
+  (wire (pts (xy 105.41 46.99) (xy 168.91 46.99))
     (stroke (width 0) (type default) (color 0 0 0 0))
   )
@@
     (stroke (width 0) (type default) (color 0 0 0 0))
   )
-  (wire (pts (xy 194.31 54.61) (xy 134.62 54.61))
-    (stroke (width 0) (type default) (color 0 0 0 0))
-  )
   (wire (pts (xy 229.87 143.51) (xy 229.87 151.13))
     (stroke (width 0) (type default) (color 0 0 0 0))
@@
     (stroke (width 0) (type default) (color 0 0 0 0))
   )
-  (wire (pts (xy 168.91 34.29) (xy 168.91 50.8))
+  (wire (pts (xy 168.91 34.29) (xy 168.91 46.99))
+    (stroke (width 0) (type default) (color 0 0 0 0))
+  )
+  (wire (pts (xy 288.29 172.72) (xy 303.53 172.72))
     (stroke (width 0) (type default) (color 0 0 0 0))
   )
@@
     (stroke (width 0) (type default) (color 0 0 0 0))
   )
+  (wire (pts (xy 294.64 177.8) (xy 303.53 177.8))
+    (stroke (width 0) (type default) (color 0 0 0 0))
+  )
   (wire (pts (xy 276.86 210.82) (xy 270.51 210.82))
     (stroke (width 0) (type default) (color 0 0 0 0))
@@
     (stroke (width 0) (type default) (color 0 0 0 0))
   )
-  (wire (pts (xy 134.62 58.42) (xy 121.92 58.42))
-    (stroke (width 0) (type default) (color 0 0 0 0))
-  )
-  (wire (pts (xy 168.91 50.8) (xy 168.91 55.88))
-    (stroke (width 0) (type default) (color 0 0 0 0))
-  )
-  (wire (pts (xy 134.62 54.61) (xy 134.62 58.42))
-    (stroke (width 0) (type default) (color 0 0 0 0))
-  )
-  (wire (pts (xy 299.72 157.48) (xy 299.72 163.83))
+  (wire (pts (xy 299.72 157.48) (xy 299.72 175.26))
     (stroke (width 0) (type default) (color 0 0 0 0))
   )
@@
     (stroke (width 0) (type default) (color 0 0 0 0))
   )
-  (wire (pts (xy 109.22 34.29) (xy 109.22 20.32))
-    (stroke (width 0) (type default) (color 0 0 0 0))
-  )
   (wire (pts (xy 111.76 154.94) (xy 125.73 154.94))
     (stroke (width 0) (type default) (color 0 0 0 0))
@@
     (stroke (width 0) (type default) (color 0 0 0 0))
   )
+  (wire (pts (xy 288.29 172.72) (xy 288.29 157.48))
+    (stroke (width 0) (type default) (color 0 0 0 0))
+  )
   (wire (pts (xy 222.25 68.58) (xy 220.98 68.58))
     (stroke (width 0) (type default) (color 0 0 0 0))
@@
     (stroke (width 0) (type default) (color 0 0 0 0))
   )
-  (wire (pts (xy 121.92 50.8) (xy 124.46 50.8))
+  (wire (pts (xy 294.64 160.02) (xy 294.64 177.8))
     (stroke (width 0) (type default) (color 0 0 0 0))
   )
@@
   (wire (pts (xy 220.98 193.04) (xy 220.98 226.06))
     (stroke (width 0) (type default) (color 0 0 0 0))
-  )
-  (wire (pts (xy 115.57 34.29) (xy 109.22 34.29))
-    (stroke (width 0) (type default) (color 0 0 0 0))
-  )
-  (label "5V" (at 130.81 50.8 0)
-    (effects (font (size 1.27 1.27)) (justify left bottom))
   )
   (label "3.3V" (at 82.55 44.45 0)
@@
     (effects (font (size 1.27 1.27)) (justify left bottom))
   )
-  (label "Vin" (at 109.22 20.32 180)
+  (label "Vin" (at 106.68 34.29 180)
     (effects (font (size 1.524 1.524)) (justify right bottom))
   )
@@
     (pin "2")
   )
-  (symbol (lib_id "power:GND") (at 299.72 163.83 0) (unit 1)
-    (in_bom yes) (on_board yes)
-    (property "Reference" "#PWR0112" (id 0) (at 299.72 170.18 0)
-      (effects (font (size 1.27 1.27)) hide)
-    )
-    (property "Value" "GND" (id 1) (at 299.72 167.64 0))
-    (property "Footprint" "" (id 2) (at 299.72 163.83 0))
-    (property "Datasheet" "" (id 3) (at 299.72 163.83 0))
+  (symbol (lib_id "power:GND") (at 299.72 184.15 0) (unit 1)
+    (in_bom yes) (on_board yes)
+    (property "Reference" "#PWR0112" (id 0) (at 299.72 190.5 0)
+      (effects (font (size 1.27 1.27)) hide)
+    )
+    (property "Value" "GND" (id 1) (at 299.72 187.96 0))
+    (property "Footprint" "" (id 2) (at 299.72 184.15 0))
+    (property "Datasheet" "" (id 3) (at 299.72 184.15 0))
     (pin "1")
   )
@@
     (property "Footprint" "" (id 2) (at 212.09 63.5 0))
     (property "Datasheet" "" (id 3) (at 212.09 63.5 0))
-    (pin "1")
-  )
-  (symbol (lib_id "power:GND") (at 129.54 53.34 0) (unit 1)
-    (in_bom yes) (on_board yes)
-    (property "Reference" "#PWR0105" (id 0) (at 129.54 59.69 0)
-      (effects (font (size 1.27 1.27)) hide)
-    )
-    (property "Value" "GND" (id 1) (at 129.54 57.15 0))
-    (property "Footprint" "" (id 2) (at 129.54 53.34 0))
-    (property "Datasheet" "" (id 3) (at 129.54 53.34 0))
     (pin "1")
   )
@@
     (pin "1")
   )
-  (symbol (lib_id "ardu_auto2_0-rescue:CONN_01X03-Arduino_shield-rescue") (at 116.84 53.34 180) (unit 1)
-    (in_bom yes) (on_board yes)
-    (property "Reference" "J5" (id 0) (at 116.84 58.42 0))
-    (property "Value" "IR_sensor" (id 1) (at 114.3 53.34 90))
-    (property "Footprint" "Connector_PinHeader_2.54mm:PinHeader_1x03_P2.54mm_Vertical" (id 2) (at 116.84 53.34 0)
-      (effects (font (size 1.27 1.27)) hide)
-    )
-    (property "Datasheet" "" (id 3) (at 116.84 53.34 0)
+  (symbol (lib_id "ardu_auto2_0-rescue:CONN_01X03-Arduino_shield-rescue") (at 308.61 175.26 0) (unit 1)
+    (in_bom yes) (on_board yes)
+    (property "Reference" "J5" (id 0) (at 308.61 170.18 0))
+    (property "Value" "IR_sensor" (id 1) (at 311.15 175.26 90))
+    (property "Footprint" "Connector_PinHeader_2.54mm:PinHeader_1x03_P2.54mm_Vertical" (id 2) (at 308.61 175.26 0)
+      (effects (font (size 1.27 1.27)) hide)
+    )
+    (property "Datasheet" "" (id 3) (at 308.61 175.26 0)
       (effects (font (size 1.27 1.27)) hide)
     )
@@
       (reference "#PWR0104") (unit 1) (value "GND") (footprint "")
     )
-    (path "/4ca52b50-ebfc-4f71-831d-caf7110bfef7"
-      (reference "#PWR0105") (unit 1) (value "GND") (footprint "")
-    )
     (path "/728904f0-d564-4241-af30-31b095b03c3b"
